File: Victor9000-RAM-Clock.kicad_sch (KiCad schematic)
At the start: 22 parts, among them U1 74LS00, U2 74LS11, U3 74LS139, U4 74LS373, U5 AS6C4008-55PCN, U6 74LS245, U7 AS6C4008-55PCN, U8 DS1315-5+, Y1 32.768 kHz

Commit message: Read and write access corrected
Parts:
- C9: footprint Capacitor_THT:CP_Radial_D4.0mm_P1.50mm -> Capacitor_THT:CP_Radial_D6.3mm_P2.50mm
Connections:
- net ~{RD}: now reaches H1.11 (RD)
- net ~{RD}: now also U5.24 (OE#), U6.1 (A->B), U7.24 (OE#), U8.12 (~{OE})
- net ~{WR}: now reaches H1.14 (~{WR})
- net ~{WR}: now also U5.29 (WE#), U7.29 (WE#), U8.3 (~{WE})
- removed net DT_~{R}: H1.12 (DT/~{R}), U5.24 (OE#), U6.1 (A->B), U7.24 (OE#), U8.12 (~{OE})
- removed net ~{SSO}: H1.7 (~{SSO}), U5.29 (WE#), U7.29 (WE#), U8.3 (~{WE})
Changed lines of the file:
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@@
   (title_block
     (title "Victor 9000 RAM Expansion")
-    (rev "v01")
+    (rev "v02")
     (comment 4 "by Florian Reitz")
   )
@@
   (no_connect (at 26.67 93.98))
   (no_connect (at 96.52 62.23))
-  (no_connect (at 26.67 116.84))
   (no_connect (at 26.67 124.46))
   (no_connect (at 26.67 129.54))
@@
   (no_connect (at 26.67 83.82))
   (no_connect (at 26.67 106.68))
-  (no_connect (at 26.67 119.38))
   (no_connect (at 26.67 76.2))
   (no_connect (at 26.67 104.14))
+  (no_connect (at 26.67 139.7))
   (no_connect (at 26.67 127))
   (no_connect (at 26.67 121.92))
   (no_connect (at 26.67 101.6))
   (no_connect (at 111.76 78.74))
+  (no_connect (at 26.67 137.16))
   (no_connect (at 261.62 57.15))
   (no_connect (at 26.67 96.52))
@@
     (stroke (width 0) (type default))
   )
+  (wire (pts (xy 21.59 119.38) (xy 26.67 119.38))
+    (stroke (width 0) (type default))
+  )
   (wire (pts (xy 128.27 38.1) (xy 134.62 38.1))
     (stroke (width 0) (type default))
@@
     (stroke (width 0) (type default))
   )
+  (wire (pts (xy 21.59 116.84) (xy 26.67 116.84))
+    (stroke (width 0) (type default))
+  )
   (wire (pts (xy 64.77 191.77) (xy 74.93 191.77))
     (stroke (width 0) (type default))
@@
     (stroke (width 0) (type default))
   )
-  (wire (pts (xy 26.67 139.7) (xy 21.59 139.7))
-    (stroke (width 0) (type default))
-  )
   (wire (pts (xy 236.22 111.76) (xy 227.33 111.76))
     (stroke (width 0) (type default))
@@
     (stroke (width 0) (type default))
   )
-  (wire (pts (xy 26.67 137.16) (xy 21.59 137.16))
-    (stroke (width 0) (type default))
-  )
   (wire (pts (xy 26.67 114.3) (xy 21.59 114.3))
     (stroke (width 0) (type default))
@@
     (effects (font (size 1.27 1.27)) (justify left bottom))
   )
-  (label "~{SSO}" (at 262.89 132.08 0) (fields_autoplaced)
+  (label "~{WR}" (at 262.89 132.08 0) (fields_autoplaced)
     (effects (font (size 1.27 1.27)) (justify left bottom))
   )
@@
     (effects (font (size 1.27 1.27)) (justify left bottom))
   )
-  (label "~{SSO}" (at 228.6 34.29 0) (fields_autoplaced)
+  (label "~{WR}" (at 228.6 34.29 0) (fields_autoplaced)
     (effects (font (size 1.27 1.27)) (justify left bottom))
   )
@@
     (effects (font (size 1.27 1.27)) (justify left bottom))
   )
-  (label "DT_~{R}" (at 21.59 139.7 0) (fields_autoplaced)
-    (effects (font (size 1.27 1.27)) (justify left bottom))
-  )
   (label "BD4" (at 175.26 34.29 0) (fields_autoplaced)
     (effects (font (size 1.27 1.27)) (justify left bottom))
@@
     (effects (font (size 1.27 1.27)) (justify left bottom))
   )
-  (label "~{SSO}" (at 21.59 137.16 0) (fields_autoplaced)
-    (effects (font (size 1.27 1.27)) (justify left bottom))
-  )
   (label "A16" (at 55.88 83.82 0) (fields_autoplaced)
     (effects (font (size 1.27 1.27)) (justify left bottom))
@@
     (effects (font (size 1.27 1.27)) (justify left bottom))
   )
-  (label "DT_~{R}" (at 262.89 129.54 0) (fields_autoplaced)
+  (label "~{RD}" (at 262.89 129.54 0) (fields_autoplaced)
     (effects (font (size 1.27 1.27)) (justify left bottom))
   )
@@
     (effects (font (size 1.27 1.27)) (justify left bottom))
   )
+  (label "~{WR}" (at 21.59 119.38 0) (fields_autoplaced)
+    (effects (font (size 1.27 1.27)) (justify left bottom))
+  )
   (label "BD6" (at 175.26 31.75 0) (fields_autoplaced)
     (effects (font (size 1.27 1.27)) (justify left bottom))
@@
     (effects (font (size 1.27 1.27)) (justify left bottom))
   )
+  (label "~{RD}" (at 21.59 116.84 0) (fields_autoplaced)
+    (effects (font (size 1.27 1.27)) (justify left bottom))
+  )
   (label "DQ6" (at 207.01 41.91 0) (fields_autoplaced)
     (effects (font (size 1.27 1.27)) (justify left bottom))
@@
     (effects (font (size 1.27 1.27)) (justify left bottom))
   )
-  (label "~{SSO}" (at 205.74 132.08 0) (fields_autoplaced)
+  (label "~{WR}" (at 205.74 132.08 0) (fields_autoplaced)
     (effects (font (size 1.27 1.27)) (justify left bottom))
   )
@@
     (effects (font (size 1.27 1.27)) (justify left bottom))
   )
-  (label "DT_~{R}" (at 205.74 129.54 0) (fields_autoplaced)
+  (label "~{RD}" (at 205.74 129.54 0) (fields_autoplaced)
     (effects (font (size 1.27 1.27)) (justify left bottom))
   )
@@
     (effects (font (size 1.27 1.27)) (justify left bottom))
   )
-  (label "DT_~{R}" (at 228.6 36.83 0) (fields_autoplaced)
+  (label "~{RD}" (at 228.6 36.83 0) (fields_autoplaced)
     (effects (font (size 1.27 1.27)) (justify left bottom))
   )
@@
     (effects (font (size 1.27 1.27)) (justify left bottom))
   )
-  (label "DT_~{R}" (at 171.45 52.07 0) (fields_autoplaced)
+  (label "~{RD}" (at 171.45 52.07 0) (fields_autoplaced)
     (effects (font (size 1.27 1.27)) (justify left bottom))
   )
@@
       (effects (font (size 1.27 1.27)) (justify left))
     )
-    (property "Footprint" "Capacitor_THT:CP_Radial_D4.0mm_P1.50mm" (at 154.6352 181.61 0)
-      (effects (font (size 1.27 1.27)) hide)
-    )
+    (property "Footprint" "Capacitor_THT:CP_Radial_D6.3mm_P2.50mm" (at 154.6352 181.61 0)
+      (effects (font (size 1.27 1.27)) hide)
+    )
